Commit message: second

File: asv_description/urdf/asv.xacro (robot description, xacro)
@@ -6,4 +6,9 @@
     <!-- Import macros -->
     <xacro:include filename="$(find asv_description)/urdf/asv_macro.xacro" />
+    <link name="base_footprint"/>
+    <joint name="base_joint" type="fixed">
+	<parent link="base_footprint"/>
+	<child link="base_link"/>
+    </joint>
     <link name="base_link">
       <visual>
@@ -12,5 +17,5 @@
           <box size="1.22 0.55 0.12"/>
         </geometry>
-	<material name="white"/>
+	<material name="burgundy"/>
       </visual>
       <collision>
@@ -44,5 +49,5 @@
     <!-- lrf -->
     <!-- front_bottom_lrf -->
-    <link name="front_bottom_lrf">
+    <link name="base_scan">
       <visual>
         <origin rpy="0 0 ${PI}" xyz="0 0 0.00"/>
@@ -54,8 +59,8 @@
     </link>
     <joint name="base_to_front_bottom_lrf" type="fixed">
-        <axis xyz="0 1 0"/>
+        <axis xyz="0 1 0" />
         <parent link="base_link"/>
-        <child link="front_bottom_lrf"/>
-        <origin xyz="0.50 0 0.45"/>
+        <child link="base_scan"/>
+        <origin xyz="0.50 0 0.45" rpy="0 0 ${PI}"/>
     </joint>
     <!-- steer -->
@@ -91,5 +96,5 @@
     -->
     <!-- rear_bottom_lrf -->
-    <link name="rear_bottom_lrf">
+    <link name="base_scan2">
       <visual>
         <origin rpy="0 0 ${PI}" xyz="0 0 0"/>
@@ -103,6 +108,6 @@
       <axis xyz="0 1 0"/>
       <parent link="base_link"/>
-      <child link="rear_bottom_lrf"/>
-      <origin  rpy="0 0 ${PI}" xyz="-0.60 0 0.45"/>
+      <child link="base_scan2"/>
+      <origin  rpy="0 0 0" xyz="-0.60 0 0.45"/>
     </joint>
     <joint name="base_to_merged_lrf" type="fixed">

File: asv_description/urdf/materials.xacro (robot description, xacro)
@@ -26,5 +26,5 @@
 </material>
 <material name="burgundy">
-  <color rgba="${50.0/255} 0.0 ${13.0/255} 1.0"/>
+  <color rgba="0.412 0.0 0.102 1.0"/>
 </material>
 </robot>

Commit message: remote

File: asv_description/urdf/asv.xacro (robot description, xacro)
@@ -10,4 +10,5 @@
 	<parent link="base_footprint"/>
 	<child link="base_link"/>
+	<origin xyz="0.38 0 0"/>
     </joint>
     <link name="base_link">
@@ -22,9 +23,22 @@
         <origin rpy="0 0 0" xyz="0 0 0.35" />
         <geometry>
-          <box size="1.0 0.55 0.4"/>
+          <box size="1.0 0.55 0.41"/>
         </geometry>
       </collision>
       <xacro:default_inertial mass="10"/>
     </link>
+    <link name="front_mark">
+	<visual>
+	    <origin xyz="0.595 0 0.36" rpy="0 0 0"/>
+	    <geometry>
+		<box size="0.08 0.08 0.08"/>
+	    </geometry>
+	    <material name="grey"/>
+	</visual>
+    </link>
+    <joint name="base_front_mark_joint" type="fixed">
+	<parent link="base_link"/>
+	<child link="front_mark"/>
+    </joint>
     <xacro:rear_wheel/>
     <xacro:front_wheel right_left="right" reflect_right_left="1"/>
